File: PCB/Miswired-Glitchy.kicad_sch (KiCad schematic)
At the start: 82 parts, among them J1 Battery Placeholder, Q3 IRLU8743PBF, SW1 DSIC08LSGET, U2 CP2102N-A02-GQFN28R, U3 LM358, U4 ESP32-S3-MINI-1-N8

Commit message: Updating some renders and docs
Accidently had the project circuit breaker docs in here
Other:
- company: True Spark Innovations -> miswired
- title: Project Circuit Breaker -> Glitchy
